Commit message: urdf updated

File: hector_small_arm_description/urdf/hector_arm_ax12_5dof.urdf.xacro (robot description, xacro)
@@ -18,5 +18,5 @@
 	<child link="connector"/>
 	<origin xyz="0 0 0.03" rpy="0 0 0" />
-	<axis xyz="0 0 1" />
+	<axis xyz="0 0 -1" />
 	<limit  lower="-1.5708" upper="1.5708" effort="10.0" velocity="1.5708" />
 <!--	<safety_controller k_position="0.1" k_velocity="1.0" soft_lower_limit="${-1.5708+0.1}" soft_upper_limit="${1.5708-0.1}" />-->
@@ -54,5 +54,5 @@
 	<parent link="endeffector_nick_link"/>
 	<child link="endeffector_yaw_link"/>
-	<origin xyz="0.0 0.035 0.0" rpy="${M_PI*0.5} ${M_PI} 0" />
+	<origin xyz="-0.1 0 0.0" rpy="${M_PI*0.5} ${M_PI} 0" />
 	<axis xyz="0 0 -1" />
 	<limit  lower="-1.5708" upper="1.5708" effort="10.0" velocity="1.5708" />
@@ -156,19 +156,34 @@
 	</inertial>
 	<visual>
-	  <origin xyz="0.0 0.0 -0.03" rpy="0 0 0" />
-	  <geometry>
-	    <mesh filename="package://hector_small_arm_description/meshes/hector_arm/hector_arm_link_0.stl"/>
-	  </geometry>
-	  <material name="red">
-	    <color rgba="1.0 0.0 0.0 1"/>
-	  </material>
-	</visual>
-        <collision>
-	  <origin xyz="0.0 0.0 -0.03" rpy="0 0 0" />
-	  <geometry>
-	    <mesh filename="package://hector_small_arm_description/meshes/hector_arm/hector_arm_link_0.stl"/>
-	  </geometry>
-	</collision>
-      </link>
+    <origin xyz="0.0 0.0 -0.03" rpy="0 0 0" />
+    <geometry>
+      <mesh filename="package://hector_small_arm_description/meshes/hector_arm/hector_arm_link_0.stl"/>
+    </geometry>
+    <material name="green">
+      <color rgba="1.0 0.0 0.0 1"/>
+    </material>
+  </visual>
+  <visual>
+    <origin xyz="-0.075 -0.03 0" rpy="${M_PI_H} 0 ${M_PI}" />
+    <geometry>
+      <mesh filename="package://hector_small_arm_description/meshes/hector_arm/hector_arm_link_0.stl"/>
+    </geometry>
+    <material name="green">
+      <color rgba="1.0 0.0 0.0 1"/>
+    </material>
+  </visual>
+  <collision>
+    <origin xyz="0.0 0.0 -0.03" rpy="0 0 0" />
+    <geometry>
+      <mesh filename="package://hector_small_arm_description/meshes/hector_arm/hector_arm_link_0.stl"/>
+    </geometry>
+  </collision>
+  <collision>
+    <origin xyz="-0.075 -0.03 0" rpy="${M_PI_H} 0 ${M_PI}" />
+    <geometry>
+      <mesh filename="package://hector_small_arm_description/meshes/hector_arm/hector_arm_link_0.stl"/>
+    </geometry>
+  </collision>
+ </link>
  <link name="endeffector_yaw_link">
 	<inertial>
@@ -182,5 +197,5 @@
 	    <mesh filename="package://hector_small_arm_description/meshes/hector_arm/hector_arm_link_4_v2.stl"/>
 	  </geometry>
-	  <material name="red">
+	  <material name="blue">
 	    <color rgba="1.0 0.0 0.0 1"/>
 	  </material>

Commit message: added fake dof for moveit

File: hector_small_arm_description/urdf/hector_arm_ax12_5dof.urdf.xacro (robot description, xacro)
@@ -60,4 +60,14 @@
 	<dynamics damping="1.0" friction="1.0"/>
       </joint>
+<!-- fake 6. dof-->
+<joint name="joint_5" type="revolute">
+  <parent link="endeffector_yaw_link"/>
+  <child link="endeffector_fake_roll_link"/>
+  <origin xyz="0.0 0.0 0.0" rpy="0 0 0" />
+  <axis xyz="1 0 0" />
+  <limit  lower="-1.5708" upper="1.5708" effort="10.0" velocity="1.5708" />
+<!--    <safety_controller k_position="0.1" k_velocity="1.0" soft_lower_limit="${-1.5708+0.1}" soft_upper_limit="${1.5708-0.1}" />-->
+  <dynamics damping="1.0" friction="1.0"/>
+</joint>
       <!-- ****** LINK DEFINITIONS ****** -->
       <link name="arm_base_link">
@@ -208,4 +218,6 @@
 	</collision>
       </link>
+  <link name="endeffector_fake_roll_link">
+  </link>
 <!-- ****** TRANSMISSION DEFINITIONS ****** -->
 	<transmission type="pr2_mechanism_model/SimpleTransmission" name="plane_trans">

Commit message: joint-2 axis corrected

File: hector_small_arm_description/urdf/hector_arm_ax12_5dof.urdf.xacro (robot description, xacro)
@@ -37,5 +37,5 @@
 	<child link="link2"/>
 	<origin xyz="0.355 0.03 0.001" rpy="0 ${M_PI} 0" />
-	<axis xyz="0 0 1" />
+	<axis xyz="0 0 -1" />
 	<limit  lower="-1.5708" upper="1.5708" effort="10.0" velocity="1.5708" />
 <!--	<safety_controller k_position="0.1" k_velocity="1.0" soft_lower_limit="${-1.5708+0.1}" soft_upper_limit="${1.5708-0.1}" />-->

Commit message: Bringup launch files for small arm. For testing on desk

File: hector_small_arm_description/urdf/hector_arm_ax12_5dof.urdf.xacro (robot description, xacro)
@@ -221,4 +221,52 @@
   </link>
 <!-- ****** TRANSMISSION DEFINITIONS ****** -->
+	<transmission name="trans_0">
+	    <type>transmission_interface/SimpleTransmission</type>
+	    <joint name="joint_0"/>
+	    <actuator name="motor_0">
+	      <hardwareInterface>JointStateInterface</hardwareInterface>
+	      <mechanicalReduction>1</mechanicalReduction>
+	    </actuator>
+ 	</transmission>
+	<transmission name="trans_1">
+	    <type>transmission_interface/SimpleTransmission</type>
+	    <joint name="joint_1"/>
+	    <actuator name="motor_1">
+	      <hardwareInterface>JointStateInterface</hardwareInterface>
+	      <mechanicalReduction>1</mechanicalReduction>
+	    </actuator>
+ 	</transmission>
+	<transmission name="trans_2">
+	    <type>transmission_interface/SimpleTransmission</type>
+	    <joint name="joint_2"/>
+	    <actuator name="motor_2">
+	      <hardwareInterface>JointStateInterface</hardwareInterface>
+	      <mechanicalReduction>1</mechanicalReduction>
+	    </actuator>
+ 	</transmission>
+	<transmission name="trans_3">
+	    <type>transmission_interface/SimpleTransmission</type>
+	    <joint name="joint_3"/>
+	    <actuator name="motor_3">
+	      <hardwareInterface>JointStateInterface</hardwareInterface>
+	      <mechanicalReduction>1</mechanicalReduction>
+	    </actuator>
+ 	</transmission>
+	<transmission name="trans_4">
+	    <type>transmission_interface/SimpleTransmission</type>
+	    <joint name="joint_4"/>
+	    <actuator name="motor_4">
+	      <hardwareInterface>JointStateInterface</hardwareInterface>
+	      <mechanicalReduction>1</mechanicalReduction>
+	    </actuator>
+ 	</transmission>
+	<transmission name="trans_5">
+	    <type>transmission_interface/SimpleTransmission</type>
+	    <joint name="joint_5"/>
+	    <actuator name="motor_5">
+	      <hardwareInterface>JointStateInterface</hardwareInterface>
+	      <mechanicalReduction>1</mechanicalReduction>
+	    </actuator>
+ 	</transmission>
 	<transmission type="pr2_mechanism_model/SimpleTransmission" name="plane_trans">
 	    <actuator name="plane_motor" />

Commit message: parameter tuning from robocup 2014 brasil. Also fixed one axis in urdf

File: hector_small_arm_description/urdf/hector_arm_ax12_5dof.urdf.xacro (robot description, xacro)
@@ -46,5 +46,5 @@
 	<child link="endeffector_nick_link"/>
 	<origin xyz="0.355 0.03 0.0" rpy="0 ${M_PI} 0" />
-	<axis xyz="0 0 -1" />
+	<axis xyz="0 0 1" />
 	<limit  lower="-1.5708" upper="1.5708" effort="10.0" velocity="1.5708" />
 <!--	<safety_controller k_position="0.1" k_velocity="1.0" soft_lower_limit="${-1.5708+0.1}" soft_upper_limit="${1.5708-0.1}" />-->
